File: telakone-robo-cpu/cpu.brd (EAGLE design)
At the start: 100 x 100 mm, 124 parts, among them K1 629105136821, X1 LIITTIMET_X3815-10, X2 MPT0.5/8-2.54, X3 MPT0.5/8-2.54, X4 MPT0.5/4-2.54, X5 MPT0.5/4-2.54, X7 MPT0.5/4-2.54

Commit message: inputs
Parts:
- removed R35: 5k90 1206, omat_ic_2:R1206
- added C31, C35: 220u 16V D, EKE:CT7343
- added C32: 10n, omat_ic_2:C0603
- added C33, C34: 2u2 50V 0805, omat_ic_2:C0805
- added C36, C37, C49: 100n, omat_ic_2:C0603
- added C38: 2u2, omat_ic_2:C0603
- added C39: 10n, cpu:OMAT_IC_2_C0603
- added C40, C41, C42, C43, C44, C45, C46, C48, C50, C51, C52, C56, C57, C59, C60: (no value), cpu:OMAT_IC_2_C0603
- added D6: LM75BD, omat_ic_2:SOIC8-N_MC
- added D7: IIS328DQTR, omat_ic_2:QFN50P400X400X100-25N
- added D8: MAX3430_SA, omat_ic_2:SOIC8-N_MC
- added D9: 74AHC14, cpu:SO14
- added L6: VLP8040-47U, omat_ic_2:VLP8040
- added N2: TPS5430DDA, omat_ic_2:SOIC8-N-EP
- added Q1, Q2, Q3, Q4: PTC, cpu:OMAT_IC_2_R1812
- added R44, R45, R46, R47, R48, R53, R54, R55, R56, R57, R60, R61, R62, R63, R64, R65, R66, R67, R68, R69, R70, R71, R72, R73, R74, R75, R76, R77, R78, R79, R80, R81, R82, R83, R84: (no value), cpu:OMAT_IC_2_R0603
- added R49: 10k0, omat_ic_2:R0603
- added R50, R85: 5k90, omat_ic_2:R0603
- added R51, R52, R59: 2k00, omat_ic_2:R0603
- added R58: 121 1206, omat_ic_2:R1206
- added V18: SK34A, omat_ic_2:DO214AC
- added V19, V20, V21, V22: ESDAXXSC6, cpu:OMAT_IC_2_SOT23-6
- added V36: SM712, omat_ic_2:SOT23
- C28: value 2u2 -> 100n
- D11: value LM75BD -> 74AHC14; device omat_ic_2:SOIC8-N_MC -> cpu:SO14
- D12: value IIS328DQTR -> 74AHC14; device omat_ic_2:QFN50P400X400X100-25N -> cpu:SO14
- L1: value VLP8040-47U -> SDR1307-15UH; device omat_ic_2:VLP8040 -> cpu:SDR1307
- R2: value 5k90 -> 3k24
- R28: value 2k00 -> 2k2; device omat_ic_2:R0603 -> cpu:OMAT_IC_2_R0603
- R29: value 2k00 -> 5k90; device omat_ic_2:R0603 -> cpu:OMAT_IC_2_R0603
- V13: value SK34A -> SBRD10200; device omat_ic_2:DO214AC -> cpu:DPACK
- moved R29 321.8 mm to (-118.0, -212.0)
- moved R28 320.0 mm to (-118.0, -209.0)
- moved C28 310.0 mm to (-118.0, -204.0)
- moved C27 305.6 mm to (-118.0, -199.0)
- moved C26 271.1 mm to (-118.0, -161.0)
- moved D11 245.0 mm to (-112.0, -180.0)
- moved D12 207.8 mm to (-112.0, -191.0)
- moved V13 197.6 mm to (-114.0, -96.0)
- moved L1 143.4 mm to (-100.0, -95.0)
Connections:
- net LEDDATA1 renamed DIR1
- net LEDDATA2 renamed DIR3
- net LEDDATA3 renamed DIR5
- net N$3 renamed USBRENUM
- net SERVO10 renamed PULSE4
- net SERVO11 renamed DIR4
- net SERVO12 renamed PULSE5
- net SERVO4 renamed PULSE0
- net SERVO5 renamed DIR0
- net SERVO6 renamed PULSE1
- net SERVO7 renamed PULSE2
- net SERVO8 renamed DIR2
- net SERVO9 renamed PULSE3
- net SERVO_PWM_6 renamed PULSE_1
- removed net N$21: V24.1, V8.C, X3.1
- removed net SERVO_PWM_10: D5.2
- removed net SERVO_PWM_11: D5.5
- removed net SERVO_PWM_12: D5.9
- removed net SERVO_PWM_4: D3.2
- removed net SERVO_PWM_5: D3.5
- removed net SERVO_PWM_7: D4.2
- removed net SERVO_PWM_8: D4.5
- removed net SERVO_PWM_9: D4.9
- removed net USART2TX1: D3.12
- removed net USART2TX2: D4.12
- removed net USART2TX3: D5.12
- new net ACCRTXHI: D8.6, R58.2, V36.1
- new net ACCRTXLO: D8.7, R58.1, V36.2
- new net DIR_0: D1.59, D3.5
- new net DIR_1: D1.60, D3.12
- new net DIR_2: D1.63, D4.5
- new net DIR_3: D1.64, D4.12
- new net DIR_4: D1.65, D5.5
- new net DIR_5: D1.66, D5.12
- new net ENABLE_N: D1.67, D2.1, D2.10, D2.13, D2.4, D3.1, D3.10, D3.13, D3.4, D4.10, D4.13, D4.4, D5.1, D5.10, D5.13, D5.4, R44.1
- new net INPUT0: R29.2, V19.1
- new net INPUT1: R54.2, V19.3
- new net INPUT10: R74.2, V21.4
- new net INPUT11: R76.2, V21.6
- new net INPUT12: R78.2, V22.1
- new net INPUT13: R80.2, V22.3
- new net INPUT14: R82.2, V22.4
- new net INPUT15: R84.2, V22.6
- new net INPUT2: R56.2, V19.4
- new net INPUT3: R60.2, V19.6
- new net INPUT4: R62.2, V20.1
- new net INPUT5: R64.2, V20.3
- new net INPUT6: R66.2, V20.4
- new net INPUT7: R68.2, V20.6
- new net INPUT8: R70.2, V21.1
- new net INPUT9: R72.2, V21.3
- new net INPUT_0: D1.98, D9.2
- new net INPUT_1: D1.99, D9.4
- new net INPUT_10: D1.116, D11.10
- new net INPUT_11: D1.117, D11.12
- new net INPUT_12: D1.118, D12.2
- new net INPUT_13: D1.119, D12.4
- new net INPUT_14: D1.122, D12.6
- new net INPUT_15: D1.123, D12.8
- new net INPUT_2: D1.111, D9.6
- new net INPUT_3: D1.112, D9.8
- new net INPUT_4: D1.113, D9.10
- new net INPUT_5: D1.7, D9.12
- new net INPUT_6: D1.8, D11.2
- new net INPUT_7: D1.9, D11.4
- new net INPUT_8: D1.114, D11.6
- new net INPUT_9: D1.115, D11.8
- new net N$38: C39.1, D9.1, R28.2, R29.1
- new net N$41: C40.1, D9.3, R53.2, R54.1
- new net N$43: C41.1, D9.5, R55.2, R56.1
- new net N$45: C42.1, D9.9, R57.2, R60.1
- new net N$47: C43.1, D9.11, R61.2, R62.1
- new net N$49: C44.1, D9.13, R63.2, R64.1
- new net N$51: C45.1, D11.1, R65.2, R66.1
- new net N$53: C46.1, D11.3, R67.2, R68.1
- new net N$55: C48.1, D11.5, R69.2, R70.1
- new net N$57: C50.1, D11.9, R71.2, R72.1
- new net N$59: C51.1, D11.11, R73.2, R74.1
- new net N$61: C52.1, D11.13, R75.2, R76.1
- new net N$63: C56.1, D12.1, R77.2, R78.1
- new net N$65: C57.1, D12.3, R79.2, R80.1
- new net N$67: C59.1, D12.5, R81.2, R82.1
- new net N$69: C60.1, D12.9, R83.2, R84.1
- new net OUT1X: Q1.1, V24.1, V8.C
- new net OUT2X: Q2.1, V10.C, V24.3
- new net OUT3X: Q3.1, V11.C, V24.4
- new net OUT4X: Q4.1, V12.C, V24.6
- new net OUT_1: D1.26, R11.1, V3.1
- new net OUT_2: D1.27, R13.1, V5.1
- new net OUT_3: R14.1, V7.1
- new net OUT_4: R15.1, V9.1
- new net PULSE_0: D1.81, D3.2
- new net PULSE_2: D1.96, D4.2
- new net PULSE_3: D1.4, D4.9
- new net PULSE_4: D1.139, D5.2
- new net PULSE_5: D1.140, D5.9
- new net SPI1MISO: D1.134
- new net SPI1MOSI: D1.135
- new net SPI1SCK: D1.133
- new net SPI_CS_PS2_N: D1.100
- new net USART1RX: D1.102, D8.1
- new net USART1TX: D1.101, D8.4
- new net USART1TXE: D1.86, D8.2, D8.3, R59.2
- net +12V: now also C33.1, C34.1, N2.7, R85.1; no longer R35.1
- net +3V3: now also C31.+, C36.1, C37.1, C38.1, C49.1, D11.14, D6.8, D7.12, D7.13, D7.14, D7.5, D8.8, D9.14, L6.2, R44.2, R49.1, R51.2, R52.2; no longer C1.+, D11.8, D12.12, D12.13, D12.5, L1.2, R1.1, R28.2, R29.2
- net +5V: now also C1.+, C35.+, L1.2, R1.1
- net GND: now also C31.-, C33.2, C34.2, C35.-, C36.2, C37.2, C38.2, C39.2, C40.2, C41.2, C42.2, C43.2, C44.2, C45.2, C46.2, C48.2, C49.2, C50.2, C51.2, C52.2, C56.2, C57.2, C59.2, C60.2, D12.7, D6.4, D6.5, D6.6, D6.7, D7.10, D7.15, D7.25, D7.4, D7.6, D7.8, D7.9, D8.5, D9.7, N2.6, N2.EP, R28.1, R45.1, R46.1, R47.1, R48.1, R50.2, R53.1, R55.1, R57.1, R59.1, R61.1, R63.1, R65.1, R67.1, R69.1, R71.1, R73.1, R75.1, R77.1, R79.1, R81.1, R83.1, V13.1, V13.3, V18.A, V19.2, V19.5, V20.2, V20.5, V21.2, V21.5, V22.2, V22.5, V36.3; no longer D11.4, D11.5, D11.6, D12.10, D12.15, D12.25, D12.4, D12.6, D12.8, D12.9, D2.1, D2.10, D2.13, D2.4, D3.1, D3.10, D3.13, D3.4, D4.10, D4.13, D4.4, D5.1, D5.10, D5.13, D5.4, V13.A
- net I2C1SCL: now also D6.2, D7.11, R52.1; no longer D11.2, D12.11, R29.1
- net I2C1SDA: now also D6.1, D7.16, R51.1; no longer D11.1, D12.16, R28.1
- net LEDDATA: now also R48.2
- net MEAS12V: now also R85.2; no longer R35.2
- net N$1: now also V13.2; no longer V13.C
- net N$17: now also C32.1, L6.1, N2.8, V18.C; no longer V12.C, V24.6, X3.7
- net N$19: now also C32.2, N2.1; no longer V11.C, V24.4, X3.5
- net N$20: now also N2.4, R49.2, R50.1; no longer V10.C, V24.3, X3.3
- net OUT1: now also Q1.2, X3.1; no longer D1.26, R11.1, V3.1
- net OUT2: now also Q2.2, X3.3; no longer D1.27, R13.1, V5.1
- net OUT3: now also Q3.2, X3.5; no longer R14.1, V7.1
- net OUT4: now also Q4.2, X3.7; no longer R15.1, V9.1
- net SERVO1: now also R45.2
- net SERVO2: now also R46.2
- net SERVO3: now also R47.2

Commit message: input liittimet, ena outputit
Parts:
- added C61: 100n, omat_ic_2:C0603
- added C62: 2u2, omat_ic_2:C0603
- added C63, C64: (no value), cpu:OMAT_IC_2_C0603
- added C65: (no value), cpu:OMAT_IC_2_C0805
- added D13, D14: 74AHCT125, cpu:SO14
- added L7: IND0603, omat_ic_2:R0603
- added L8: IND0603, cpu:OMAT_IC_2_R0603
- added R35, R86, R87, R88, R89, R90, R91, R92, R93, R94, R95, R96: (no value), cpu:OMAT_IC_2_R0603
- added V23, V25: ESDAXXSC6, cpu:OMAT_IC_2_SOT23-6
- added X10, X9: MPT0.5/8-2.54, cpu:OMAT_IC_2_MPT0.5/8-2.54
- added X11, X12, X13, X14: MPT0.5/4-2.54, cpu:MPT0.5/4-2.54
- added X8: PS-JOYSTICK, cpu:PS-JOYSTICK
- added Y1, Y2, Y3, Y4: PTH2.6-5.5SQ, EKE:PTH-2.6-5.5SQ
- moved X2 162.1 mm to (91.4, 71.2), turned to 90 degrees
- moved X6 159.7 mm to (93.2, 21.0), turned to 90 degrees
- moved F1 156.0 mm to (87.4, 8.62)
- moved X7 128.4 mm to (57.3, 94.5), turned to 180 degrees
- moved X3 120.4 mm to (83.0, 95.5), turned to 180 degrees
- moved X5 104.5 mm to (43.9, 94.5), turned to 180 degrees
- moved D1 84.1 mm to (51.9, 51.2)
- moved X4 79.2 mm to (28.4, 94.5), turned to 180 degrees
Connections:
- removed net SPI1SCK: D1.133
- new net ENA0: R89.2, V23.1, X11.1
- new net ENA1: R90.2, V23.3, X11.2
- new net ENA2: R91.2, V23.4, X11.3
- new net ENA3: R92.2, V23.6, X11.4
- new net ENA4: R93.2, V25.1, X12.1
- new net ENA5: R94.2, V25.3, X12.2
- new net ENA_0: D1.56, D13.2
- new net ENA_1: D1.57, D13.5
- new net ENA_2: D1.87, D13.9
- new net ENA_3: D1.88, D13.12
- new net ENA_4: D1.89, D14.2
- new net ENA_5: D1.90, D14.5
- new net I2CVCC: C65.1, L8.1, X14.1
- new net N$21: R86.1, X8.2
- new net N$3: R35.1, X8.1
- new net N$39: R87.1, X8.6
- new net N$42: R88.1, X8.7
- new net N$44: D13.3, R89.1
- new net N$46: D13.6, R90.1
- new net N$48: D13.8, R91.1
- new net N$50: D13.11, R92.1
- new net N$52: D14.3, R93.1
- new net N$54: D14.6, R94.1
- new net N$56: D14.8, R95.1
- new net N$58: D14.11, R96.1
- new net N$60: X14.2
- new net N$62: X14.4
- new net PSVCC: C61.1, C62.1, L7.1, X8.5
- new net SPARE1: R95.2, V25.4, X12.3
- new net SPARE2: R96.2, V25.6, X12.4
- new net SPARE_1: D1.91, D14.9
- new net SPARE_2: D1.92, D14.12
- new net SPI1CLK: D1.133, R88.2
- net +12V: now also X13.1, X13.2, X13.3, X13.4
- net +3V3: now also L7.2
- net +5V: now also C63.1, C64.1, D13.14, D14.14, L8.2
- net ENABLE_N: now also D13.1, D13.10, D13.13, D13.4, D14.10, D14.13, D14.4
- net GND: now also C61.2, C62.2, C63.2, C64.2, C65.2, D13.7, D14.7, V23.2, V23.5, V25.2, V25.5, X14.3, X8.4, Y1.1, Y2.1, Y3.1, Y4.1
- net INPUT0: now also X9.1
- net INPUT1: now also X9.2
- net INPUT10: now also X10.3
- net INPUT11: now also X10.4
- net INPUT12: now also X10.5
- net INPUT13: now also X10.6
- net INPUT14: now also X10.7
- net INPUT15: now also X10.8
- net INPUT2: now also X9.3
- net INPUT3: now also X9.4
- net INPUT4: now also X9.5
- net INPUT5: now also X9.6
- net INPUT6: now also X9.7
- net INPUT7: now also X9.8
- net INPUT8: now also X10.1
- net INPUT9: now also X10.2
- net SPI1MISO: now also R35.2
- net SPI1MOSI: now also R86.2
- net SPI_CS_PS2_N: now also R87.2

Commit message: i2c expander yms
Parts:
- added C66, C67: (no value), cpu:OMAT_IC_2_C0805
- added D15: PCA9517, cpu:OMAT_IC_2_SOIC8-N_MC
- added L9: IND0603, cpu:OMAT_IC_2_R0603
- added R100, R99: 2k00, omat_ic_2:R0603
- added X15: MPT0.5/4-2.54, cpu:MPT0.5/4-2.54
- moved L8 49.6 mm to (-126.0, -530.0)
Connections:
- removed net N$60: X14.2
- removed net N$62: X14.4
- new net I2CSCL: D15.7, R100.1, X14.4
- new net I2CSDA: D15.6, R99.1, X14.2
- net +3V3: now also C67.1, D15.1, L8.2
- net +5V: now also L9.1; no longer L8.2
- net ACCRTXHI: now also X15.3
- net ACCRTXLO: now also X15.4
- net GND: now also C66.2, C67.2, D12.11, D12.13, D15.4
- net I2C1SCL: now also D15.2
- net I2C1SDA: now also D15.3
- net I2CVCC: now also C66.1, D15.5, D15.8, L9.2, R100.2, R99.2
- net OUT_3: now also D1.69
- net OUT_4: now also D1.70
- net SERVO_PWM_3: now also D1.46

Commit message: finish schematics, rough initial placement
Parts:
- added C68, C69: (no value), cpu:OMAT_IC_2_C0805
- added V26: SRV05-4, cpu:OMAT_IC_2_SOT23-6
- added V27: ESDAXXSC6, cpu:OMAT_IC_2_SOT23-6
- moved L8 594.2 mm to (16.0, 47.0)
- moved L9 591.3 mm to (16.0, 49.0)
- moved X15 572.0 mm to (4.00, 38.0), turned to 270 degrees
- moved R100 571.4 mm to (14.0, 42.0)
- moved R99 565.8 mm to (11.0, 42.0)
- moved R96 564.5 mm to (87.0, 57.0)
- moved R93 563.1 mm to (87.0, 63.0)
- moved R94 559.9 mm to (87.0, 61.0)
- moved V25 559.4 mm to (90.0, 60.0)
- moved R95 556.6 mm to (87.0, 59.0)
- moved C67 555.8 mm to (21.0, 42.0)
- moved R90 553.9 mm to (86.0, 49.0)
- moved C64 551.9 mm to (82.0, 59.0), turned to 90 degrees
- moved C65 551.1 mm to (11.0, 50.0)
- moved C66 550.9 mm to (17.0, 42.0)
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Connections:
- new net SERVO_VCC1: C68.1
- new net SERVO_VCC2: C69.1
- net GND: now also C68.2, C69.2, V26.2, V27.2, V27.5
- net I2CSCL: now also V27.4
- net I2CSDA: now also V27.3
- net I2CVCC: now also V27.1
- net USB_DM: now also V26.4
- net USB_DP: now also V26.3
- net VUSB: now also V26.5

Commit message: signals routed, almost
Parts:
- added X16: MPT0.5/4-2.54, cpu:MPT0.5/4-2.54
- moved R45 53.0 mm to (6.25, 64.8), flipped to the bottom, turned to 90 degrees
- moved K1 52.5 mm to (78.5, 4.00)
- moved R7 49.8 mm to (71.5, 19.2)
- moved X1 47.3 mm to (48.2, 60.5), turned to 180 degrees
- moved R6 47.0 mm to (71.5, 20.8), turned to 180 degrees
- moved R46 45.9 mm to (6.25, 57.2), flipped to the bottom, turned to 90 degrees
- moved C7 45.8 mm to (9.50, 70.8), turned to 90 degrees
- moved R85 45.1 mm to (89.2, 68.5)
- moved R36 45.0 mm to (89.2, 66.8)
- moved L5 44.4 mm to (12.2, 69.0)
- moved X2 43.0 mm to (4.00, 69.0)
- moved C68 42.6 mm to (9.50, 67.2), turned to 270 degrees
- moved R5 41.3 mm to (71.5, 22.2)
- moved R22 41.0 mm to (9.00, 64.2), turned to 180 degrees
- moved R47 40.8 mm to (6.25, 49.5), flipped to the bottom, turned to 90 degrees
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Connections:
- removed net SERVO_VCC1: C68.1
- removed net SERVO_VCC2: C69.1
- new net ENABLE_PWM_N: D1.124, D2.1, D2.10, D2.13, D2.4
- net ACCRTXHI: now also V36.2; no longer V36.1
- net ACCRTXLO: now also V36.1; no longer V36.2
- net DIR0: now also V14.4; no longer V14.3
- net DIR1: now also V14.1; no longer V14.6
- net DIR2: now also V15.4; no longer V15.3
- net DIR3: now also V15.1; no longer V15.6
- net DIR4: now also V17.4; no longer V17.3
- net DIR5: now also V17.1; no longer V17.6
- net ENA0: now also V23.6; no longer V23.1
- net ENA1: now also V23.4; no longer V23.3
- net ENA2: now also V23.3; no longer V23.4
- net ENA3: now also V23.1; no longer V23.6
- net ENA4: now also V25.6; no longer V25.1
- net ENA5: now also V25.4; no longer V25.3
- net ENABLE_N: now also D14.1, D4.1; no longer D2.1, D2.10, D2.13, D2.4
- net GND: now also X16.1, X16.4, X2.3, X2.6; no longer X2.5, X2.8
- net I2CSCL: now also V27.3; no longer V27.4
- net I2CSDA: now also V27.4; no longer V27.3
- net I2CVCC: now also V27.6; no longer V27.1
- net INPUT0: now also V19.3; no longer V19.1
- net INPUT1: now also V19.1; no longer V19.3
- net INPUT10: now also V21.6; no longer V21.4
- net INPUT11: now also V21.4; no longer V21.6
- net INPUT12: now also V22.3; no longer V22.1
- net INPUT13: now also V22.1; no longer V22.3
- net INPUT14: now also V22.6; no longer V22.4
- net INPUT15: now also V22.4; no longer V22.6
- net INPUT2: now also V19.6; no longer V19.4
- net INPUT3: now also V19.4; no longer V19.6
- net INPUT4: now also V20.3; no longer V20.1
- net INPUT5: now also V20.1; no longer V20.3
- net INPUT6: now also V20.6; no longer V20.4
- net INPUT7: now also V20.4; no longer V20.6
- net INPUT8: now also V21.3; no longer V21.1
- net INPUT9: now also V21.1; no longer V21.3
- net LEDDATA: now also V6.1, X16.3; no longer V6.6, X2.7
- net LED_VCC: now also C69.1, X16.2; no longer X2.6
- net PULSE0: now also V14.6; no longer V14.1
- net PULSE1: now also V14.3; no longer V14.4
- net PULSE2: now also V15.6; no longer V15.1
- net PULSE3: now also V15.3; no longer V15.4
- net PULSE4: now also V17.6; no longer V17.1
- net PULSE5: now also V17.3; no longer V17.4
- net SERVO1: now also V6.6; no longer V6.1
- net SERVO2: now also V6.4, X2.5; no longer V6.3, X2.3
- net SERVO3: now also V6.3, X2.8; no longer V6.4, X2.4
- net SERVO_VCC: now also C68.1, X2.4, X2.7
- net SPARE1: now also V25.3; no longer V25.4
- net SPARE2: now also V25.1; no longer V25.6
- net SPI_CS_PS2_N: now also D1.35; no longer D1.100
Routing:
- net ENABLE_N: track 0.00 -> 192.4 mm
- net USART1TX: track 0.00 -> 142.1 mm, vias 0 -> 2
- net USART1RX: track 0.00 -> 140.6 mm, vias 0 -> 2
- net USART1TXE: track 0.00 -> 137.3 mm, vias 0 -> 2
- net SERVO_PWM_3: track 0.00 -> 118.3 mm, vias 0 -> 2
- net SERVO_PWM_2: track 0.00 -> 117.6 mm, vias 0 -> 2
- net SERVO_PWM_1: track 0.00 -> 109.4 mm, vias 0 -> 2
- net USART2TX: track 0.00 -> 103.7 mm, vias 0 -> 2
- net OUT_1: track 0.00 -> 92.5 mm, vias 0 -> 3
- net OUT_2: track 0.00 -> 89.6 mm, vias 0 -> 3
- net INPUT_6: track 0.00 -> 77.2 mm, vias 0 -> 3
- net OUT_3: track 0.00 -> 77.0 mm, vias 0 -> 3
- net INPUT_7: track 0.00 -> 74.3 mm, vias 0 -> 3
- net OUT_4: track 0.00 -> 72.3 mm, vias 0 -> 3
- net USB_DP: track 0.00 -> 70.5 mm, vias 0 -> 2
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
Commit message: routed
Parts:
- removed F1: KEYSTONE-3549-2, omat_ic_2:KEYSTONE-3549-2
- added F2: MINIBLADE-FUSEHOLDER-3568, cpu:KEYSTONE-3568
- added X17: MPT0.5/4-2.54, cpu:MPT0.5/4-2.54
- moved R36 40.9 mm to (50.8, 80.5), turned to 180 degrees
- moved R85 40.9 mm to (50.8, 82.2), turned to 180 degrees
- moved V16 22.3 mm to (77.9, 88.0), turned to 270 degrees
- moved L7 19.0 mm to (35.5, 9.25)
- moved R44 11.5 mm to (72.8, 33.8), turned to 90 degrees
- moved C62 4.78 mm to (50.8, 1.50), turned to 180 degrees
- moved C13 4.56 mm to (53.8, 51.0), turned to 315 degrees
- moved R50 4.16 mm to (36.5, 59.5), turned to 270 degrees
- moved C61 2.50 mm to (50.8, 6.25)
- moved C16 2.14 mm to (42.8, 38.0), turned to 135 degrees
- moved C58 1.46 mm to (47.0, 41.2), turned to 225 degrees
- moved R49 1.25 mm to (35.8, 61.8)
- moved C17 0.90 mm to (56.8, 44.5), turned to 315 degrees
- moved C32 0.75 mm to (32.8, 67.0)
- moved C4 0.75 mm to (81.2, 74.2)
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Connections:
- net N$1 renamed PH5V
- net N$17 renamed PH3V3
- net N$19 renamed BOOT3V3
- net N$2 renamed BOOT5V
- removed net N$8: F1.2, F1.3, X6.2
- new net 12VIN: F2.1, F2.4, X6.2
- net +12V: now also F2.2, F2.3; no longer F1.1, F1.4
- net GND: now also X17.1, X17.2, X17.3, X17.4
Routing:
- net +3V3: track 22.3 -> 458.3 mm, vias 3 -> 31
- net +5V: track 12.6 -> 233.2 mm, vias 0 -> 15
- net MEAS12V: track 0.00 -> 88.1 mm, vias 0 -> 2
- net +12V: track 45.6 -> 122.1 mm
- net GND: track 70.4 -> 13.6 mm, vias 0 -> 235
- net SERVO_VCC: track 11.9 -> 33.7 mm
- net PH5V: track 0.00 -> 19.4 mm, vias 0 -> 1
- net PSVCC: track 7.69 -> 24.7 mm
- net I2CVCC: track 27.2 -> 38.7 mm, vias 0 -> 2
- net 12VIN: track 0.00 -> 10.9 mm
- net PH3V3: track 0.00 -> 9.37 mm, vias 0 -> 1
- net N$20: track 0.00 -> 5.53 mm
- net N$4: track 0.00 -> 3.79 mm
- net BOOT5V: track 0.00 -> 3.32 mm, vias 0 -> 1
- net BOOT3V3: track 0.00 -> 2.99 mm, vias 0 -> 1
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- added copper zone on layer 1, net 12VIN
- added copper zone on layer 1, net GND
- added copper zone on layer 16, net GND

Commit message: Final v1
Parts:
- added U$1: DAFUG, telakone-aux-gps:DAFUG
- moved C9 1.34 mm to (68.2, 34.5)
- moved R44 0.56 mm to (73.0, 33.2)
- moved C18 0.16 mm to (49.9, 44.9)
- renumbered F2 to F1, K1 to X18
Routing:
- net +3V3: track 458.3 -> 463.3 mm
- net VCAP1: track 2.97 -> 1.69 mm
- net OUT_3: track 77.0 -> 77.6 mm
- net ENA_0: track 34.9 -> 34.3 mm
- net ENA_1: track 37.5 -> 37.0 mm
- net ENABLE_N: track 194.4 -> 193.9 mm
- net GND: vias 235 -> 260
Other:
- board text added: "6+3 AXIS ROBOT ARM CONTROLLER"
- board text added: "DBG"
- board text added: "ERR"
- board text added: "FUSE 2A"
- board text added: "KIMMOLI 2018"
- board text added: "RUN"
- board text added: "TELAKONE"
- board text added: "X"
- board text added: "Y"
- board text added: "Z"
