File: telakone-robo-cpu/cpu.sch (EAGLE design)
At the start: 252 parts, among them K1 629105136821, Q1 PTC, Q2 PTC, Q3 PTC, Q4 PTC, X1 LIITTIMET_X3815-10, X10 MPT0.5/8-2.54, X11 MPT0.5/4-2.54, X12 MPT0.5/4-2.54, X13 MPT0.5/4-2.54, X14 MPT0.5/4-2.54, X15 MPT0.5/4-2.54, X16 MPT0.5/4-2.54, X2 MPT0.5/8-2.54, X3 MPT0.5/8-2.54, X4 MPT0.5/4-2.54, X5 MPT0.5/4-2.54, X7 MPT0.5/4-2.54, X8 PS-JOYSTICK, X9 MPT0.5/8-2.54, Y1 PTH2.6-5.5SQ, Y2 PTH2.6-5.5SQ, Y3 PTH2.6-5.5SQ, Y4 PTH2.6-5.5SQ

Commit message: routed
Parts:
- removed F1: KEYSTONE-3549-2, omat_ic_2:KEYSTONE-3549-2
- added F2: MINIBLADE-FUSEHOLDER-3568, cpu:MINIBLADE-FUSEHOLDER-3568
- added X17: MPT0.5/4-2.54, cpu:MPT0.5/4-2.54
Connections:
- net N$1 renamed PH5V
- net N$17 renamed PH3V3
- net N$19 renamed BOOT3V3
- net N$2 renamed BOOT5V
- removed net N$8: F1.2, X6.2
- new net 12VIN: F2.1, X6.2
- net +12V: now also F2.2; no longer F1.1
- net GND: now also X17.1, X17.2, X17.3, X17.4
Other:
- moved on the sheet: V16
Changed lines of the file:
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@@
 <part name="X6" library="omat_ic_2" deviceset="TE_RUUVILIITIN2" device=""/>
 <part name="GND10" library="EKE" deviceset="GND" device=""/>
-<part name="F1" library="omat_ic_2" deviceset="KEYSTONE-3549-2" device=""/>
 <part name="V16" library="omat_ic_2" deviceset="SMAJXXA" device="" value="SMAJ20A"/>
 <part name="P+10" library="EKE" deviceset="+12V" device=""/>
@@
 <part name="X16" library="cpu" deviceset="MPT0.5/4-2.54" device=""/>
 <part name="X2" library="cpu" deviceset="MPT0.5/8-2.54" device=""/>
+<part name="F2" library="cpu" deviceset="MINIBLADE-FUSEHOLDER" device="-3568"/>
+<part name="X17" library="cpu" deviceset="MPT0.5/4-2.54" device=""/>
+<part name="GND129" library="cpu" deviceset="GND" device=""/>
 </parts>
 <sheets>
@@
 <attribute name="VALUE" x="134.62" y="180.34" size="1.778" layer="96"/>
 </instance>
-<instance part="P+9" gate="1" x="101.6" y="213.36" smashed="yes">
-<attribute name="VALUE" x="99.06" y="208.28" size="1.778" layer="96" rot="R90"/>
+<instance part="P+9" gate="1" x="119.38" y="213.36" smashed="yes">
+<attribute name="VALUE" x="116.84" y="208.28" size="1.778" layer="96" rot="R90"/>
 </instance>
 <instance part="D10" gate="G$1" x="198.12" y="73.66" smashed="yes">
@@
 <attribute name="VALUE" x="66.04" y="180.34" size="1.778" layer="96"/>
 </instance>
-<instance part="F1" gate="G$1" x="88.9" y="205.74" smashed="yes" rot="MR0">
-<attribute name="NAME" x="92.71" y="207.137" size="1.778" layer="95" rot="MR0"/>
-<attribute name="VALUE" x="92.71" y="202.819" size="1.778" layer="96" rot="MR0"/>
-</instance>
-<instance part="V16" gate="G$1" x="99.06" y="195.58" smashed="yes" rot="R90">
-<attribute name="NAME" x="97.155" y="193.802" size="1.778" layer="95" rot="R90"/>
-<attribute name="VALUE" x="102.489" y="193.802" size="1.778" layer="96" rot="R90"/>
+<instance part="V16" gate="G$1" x="116.84" y="195.58" smashed="yes" rot="R90">
+<attribute name="NAME" x="114.935" y="193.802" size="1.778" layer="95" rot="R90"/>
+<attribute name="VALUE" x="120.269" y="193.802" size="1.778" layer="96" rot="R90"/>
 </instance>
 <instance part="N2" gate="G$1" x="193.04" y="142.24" smashed="yes">
@@
 <attribute name="VALUE" x="60.96" y="48.26" size="1.778" layer="96"/>
 </instance>
+<instance part="F2" gate="G$1" x="88.9" y="205.74" smashed="yes">
+<attribute name="NAME" x="85.09" y="207.137" size="1.778" layer="95"/>
+<attribute name="VALUE" x="72.39" y="202.819" size="1.778" layer="96"/>
+</instance>
 </instances>
 <busses>
 </busses>
 <nets>
-<net name="N$1" class="0">
+<net name="PH5V" class="0">
 <segment>
 <pinref part="N1" gate="G$1" pin="PH"/>
@@
 <pinref part="L1" gate="G$1" pin="1"/>
 <pinref part="V13" gate="G$1" pin="C"/>
+<label x="218.44" y="205.74" size="1.778" layer="95"/>
 </segment>
 </net>
-<net name="N$2" class="0">
+<net name="BOOT5V" class="0">
 <segment>
 <pinref part="N1" gate="G$1" pin="BOOT"/>
@@
 <pinref part="V16" gate="G$1" pin="A"/>
 <wire x1="68.58" y1="187.96" x2="68.58" y2="185.42" width="0.1524" layer="91"/>
-<wire x1="99.06" y1="193.04" x2="99.06" y2="187.96" width="0.1524" layer="91"/>
-<wire x1="99.06" y1="187.96" x2="68.58" y2="187.96" width="0.1524" layer="91"/>
+<wire x1="116.84" y1="193.04" x2="116.84" y2="187.96" width="0.1524" layer="91"/>
+<wire x1="116.84" y1="187.96" x2="68.58" y2="187.96" width="0.1524" layer="91"/>
 <junction x="68.58" y="187.96"/>
 <pinref part="X6" gate="G$1" pin="1"/>
@@
 <wire x1="154.94" y1="200.66" x2="154.94" y2="205.74" width="0.1524" layer="91"/>
 <junction x="154.94" y="205.74"/>
-<wire x1="137.16" y1="205.74" x2="101.6" y2="205.74" width="0.1524" layer="91"/>
+<wire x1="137.16" y1="205.74" x2="119.38" y2="205.74" width="0.1524" layer="91"/>
 <junction x="137.16" y="205.74"/>
-<wire x1="101.6" y1="205.74" x2="101.6" y2="210.82" width="0.1524" layer="91"/>
+<wire x1="119.38" y1="205.74" x2="119.38" y2="210.82" width="0.1524" layer="91"/>
 <pinref part="P+9" gate="1" pin="+12V"/>
-<pinref part="F1" gate="G$1" pin="1"/>
-<wire x1="101.6" y1="205.74" x2="99.06" y2="205.74" width="0.1524" layer="91"/>
-<junction x="101.6" y="205.74"/>
+<wire x1="119.38" y1="205.74" x2="116.84" y2="205.74" width="0.1524" layer="91"/>
+<junction x="119.38" y="205.74"/>
 <pinref part="V16" gate="G$1" pin="C"/>
-<wire x1="99.06" y1="205.74" x2="93.98" y2="205.74" width="0.1524" layer="91"/>
-<wire x1="99.06" y1="198.12" x2="99.06" y2="205.74" width="0.1524" layer="91"/>
-<junction x="99.06" y="205.74"/>
+<wire x1="116.84" y1="205.74" x2="93.98" y2="205.74" width="0.1524" layer="91"/>
+<wire x1="116.84" y1="198.12" x2="116.84" y2="205.74" width="0.1524" layer="91"/>
+<junction x="116.84" y="205.74"/>
+<pinref part="F2" gate="G$1" pin="2"/>
 </segment>
 <segment>
@@
 </segment>
 </net>
-<net name="N$8" class="0">
+<net name="12VIN" class="0">
 <segment>
-<pinref part="F1" gate="G$1" pin="2"/>
 <pinref part="X6" gate="G$1" pin="2"/>
 <wire x1="83.82" y1="205.74" x2="63.5" y2="205.74" width="0.1524" layer="91"/>
+<pinref part="F2" gate="G$1" pin="1"/>
+<label x="71.12" y="205.74" size="1.778" layer="95"/>
 </segment>
 </net>
-<net name="N$17" class="0">
+<net name="PH3V3" class="0">
 <segment>
 <pinref part="N2" gate="G$1" pin="PH"/>
@@
 <wire x1="228.6" y1="144.78" x2="228.6" y2="149.86" width="0.1524" layer="91"/>
 <junction x="228.6" y="149.86"/>
+<label x="218.44" y="149.86" size="1.778" layer="95"/>
 </segment>
 </net>
-<net name="N$19" class="0">
+<net name="BOOT3V3" class="0">
 <segment>
 <pinref part="N2" gate="G$1" pin="BOOT"/>
@@
 <attribute name="NAME" x="372.11" y="153.162" size="1.778" layer="95" rot="MR0"/>
 </instance>
+<instance part="X17" gate="G$1" x="373.38" y="68.58" smashed="yes" rot="MR0">
+<attribute name="VALUE" x="372.11" y="66.04" size="1.778" layer="96" rot="MR0"/>
+<attribute name="NAME" x="372.11" y="82.042" size="1.778" layer="95" rot="MR0"/>
+</instance>
+<instance part="GND129" gate="1" x="342.9" y="63.5" smashed="yes">
+<attribute name="VALUE" x="340.36" y="60.96" size="1.778" layer="96"/>
+</instance>
 </instances>
 <busses>
@@
 <pinref part="GND119" gate="1" pin="GND"/>
 </segment>
+<segment>
+<pinref part="X17" gate="G$1" pin="1"/>
+<wire x1="363.22" y1="78.74" x2="342.9" y2="78.74" width="0.1524" layer="91"/>
+<wire x1="342.9" y1="78.74" x2="342.9" y2="76.2" width="0.1524" layer="91"/>
+<pinref part="X17" gate="G$1" pin="4"/>
+<wire x1="342.9" y1="76.2" x2="342.9" y2="73.66" width="0.1524" layer="91"/>
+<wire x1="342.9" y1="73.66" x2="342.9" y2="71.12" width="0.1524" layer="91"/>
+<wire x1="342.9" y1="71.12" x2="342.9" y2="66.04" width="0.1524" layer="91"/>
+<wire x1="363.22" y1="71.12" x2="342.9" y2="71.12" width="0.1524" layer="91"/>
+<junction x="342.9" y="71.12"/>
+<pinref part="X17" gate="G$1" pin="3"/>
+<wire x1="363.22" y1="73.66" x2="342.9" y2="73.66" width="0.1524" layer="91"/>
+<junction x="342.9" y="73.66"/>
+<pinref part="X17" gate="G$1" pin="2"/>
+<wire x1="363.22" y1="76.2" x2="342.9" y2="76.2" width="0.1524" layer="91"/>
+<junction x="342.9" y="76.2"/>
+<pinref part="GND129" gate="1" pin="GND"/>
+</segment>
 </net>

Commit message: Final v1
Parts:
- added U$1: DAFUG, telakone-aux-gps:DAFUG
- renumbered F2 to F1, K1 to X18
Changed lines of the file:
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@@
 <part name="V1" library="cpu" deviceset="2N3904" device=""/>
 <part name="R21" library="aux-io" deviceset="PASSIIVIT_RES" device="0603" value="1k47"/>
-<part name="K1" library="cpu" deviceset="629105136821" device=""/>
+<part name="X18" library="cpu" deviceset="629105136821" device=""/>
 <part name="GND6" library="EKE" deviceset="GND" device=""/>
 <part name="FRAME5" library="cpu" deviceset="AUX-IO_OMAT_DINA3_L" device=""/>
@@
 <part name="X16" library="cpu" deviceset="MPT0.5/4-2.54" device=""/>
 <part name="X2" library="cpu" deviceset="MPT0.5/8-2.54" device=""/>
-<part name="F2" library="cpu" deviceset="MINIBLADE-FUSEHOLDER" device="-3568"/>
+<part name="F1" library="cpu" deviceset="MINIBLADE-FUSEHOLDER" device="-3568"/>
 <part name="X17" library="cpu" deviceset="MPT0.5/4-2.54" device=""/>
 <part name="GND129" library="cpu" deviceset="GND" device=""/>
+<part name="U$1" library="telakone-aux-gps" deviceset="DAFUG" device=""/>
 </parts>
 <sheets>
@@
 <attribute name="VALUE" x="60.96" y="48.26" size="1.778" layer="96"/>
 </instance>
-<instance part="F2" gate="G$1" x="88.9" y="205.74" smashed="yes">
+<instance part="F1" gate="G$1" x="88.9" y="205.74" smashed="yes">
 <attribute name="NAME" x="85.09" y="207.137" size="1.778" layer="95"/>
 <attribute name="VALUE" x="72.39" y="202.819" size="1.778" layer="96"/>
@@
 <wire x1="116.84" y1="198.12" x2="116.84" y2="205.74" width="0.1524" layer="91"/>
 <junction x="116.84" y="205.74"/>
-<pinref part="F2" gate="G$1" pin="2"/>
+<pinref part="F1" gate="G$1" pin="2"/>
 </segment>
 <segment>
@@
 <pinref part="X6" gate="G$1" pin="2"/>
 <wire x1="83.82" y1="205.74" x2="63.5" y2="205.74" width="0.1524" layer="91"/>
-<pinref part="F2" gate="G$1" pin="1"/>
+<pinref part="F1" gate="G$1" pin="1"/>
 <label x="71.12" y="205.74" size="1.778" layer="95"/>
 </segment>
@@
 <attribute name="VALUE" x="66.802" y="118.11" size="1.778" layer="96" rot="R90"/>
 </instance>
-<instance part="K1" gate="G$1" x="27.94" y="172.72" smashed="yes" rot="MR0">
+<instance part="X18" gate="G$1" x="27.94" y="172.72" smashed="yes" rot="MR0">
 <attribute name="NAME" x="35.56" y="186.69" size="1.778" layer="95" rot="MR0"/>
 <attribute name="VALUE" x="35.56" y="167.64" size="1.778" layer="96" rot="MR0"/>
@@
 <attribute name="VALUE" x="68.58" y="208.28" size="1.778" layer="96"/>
 </instance>
+<instance part="U$1" gate="G$1" x="274.32" y="7.62" smashed="yes"/>
 </instances>
 <busses>
@@
 </segment>
 <segment>
-<pinref part="K1" gate="G$1" pin="5"/>
+<pinref part="X18" gate="G$1" pin="5"/>
 <wire x1="38.1" y1="172.72" x2="43.18" y2="172.72" width="0.1524" layer="91"/>
 <pinref part="GND6" gate="1" pin="GND"/>
@@
 <label x="50.8" y="180.34" size="1.778" layer="95"/>
 <wire x1="127" y1="180.34" x2="38.1" y2="180.34" width="0.1524" layer="91"/>
-<pinref part="K1" gate="G$1" pin="2"/>
+<pinref part="X18" gate="G$1" pin="2"/>
 </segment>
 <segment>
@@
 <wire x1="48.26" y1="177.8" x2="38.1" y2="177.8" width="0.1524" layer="91"/>
 <junction x="48.26" y="177.8"/>
-<pinref part="K1" gate="G$1" pin="3"/>
+<pinref part="X18" gate="G$1" pin="3"/>
 </segment>
 <segment>
@@
 <wire x1="76.2" y1="182.88" x2="38.1" y2="182.88" width="0.1524" layer="91"/>
 <label x="50.8" y="182.88" size="1.778" layer="95"/>
-<pinref part="K1" gate="G$1" pin="1"/>
+<pinref part="X18" gate="G$1" pin="1"/>
 <pinref part="V26" gate="G$1" pin="VCC"/>
 <wire x1="68.58" y1="226.06" x2="76.2" y2="226.06" width="0.1524" layer="91"/>
